File: Hardware/MotorDriver.sch (KiCad schematic (older format))
At the start: 58 parts, among them J1 Prog, J10 perif_pins, J11 STEPPER1, J12 STEPPER2, J2 Conn_01x05, J3 SERIAL, J4 MOTOROUTPUT, J5 I2C, J6 ENCODER2, J7 perif_vcc, J8 ENCODER1, J9 perif_gnd, Q1 IPD068P03, SW1 SW_DIP_x01, U1 DRV8870DDA, U2 L7805, U3 DRV8870DDA, U4 AT90CAN128-16AU, U5 MCP2551-I-SN, Y1 OSCILLATOR-16MHZ

Commit message: Readme and pictures
Parts:
- Y1: symbol SparkFun-Clocks:OSCILLATOR-16MHZSMD-7X5-4PAD -> MotorDriver-rescue:OSCILLATOR-16MHZSMD-7X5-4PAD-SparkFun-Clocks
Changed lines of the file:
@@
 EESchema Schematic File Version 4
 LIBS:MotorDriver-cache
-EELAYER 26 0
+EELAYER 29 0
 EELAYER END
 $Descr A4 11693 8268
@@
 $EndComp
 $Comp
-L SparkFun-Clocks:OSCILLATOR-16MHZSMD-7X5-4PAD Y1
+L MotorDriver-rescue:OSCILLATOR-16MHZSMD-7X5-4PAD-SparkFun-Clocks Y1
 U 1 1 5BA6A03A
 P 1350 1000
